Commit message: Add multi-robot support with launch files and RViz configurations
- Created .gitignore for build artifacts and IDE files.
- Updated CMakeLists.txt to install RViz files.
- Enhanced multi_robot.launch.py to include static transforms for multiple robots.
- Added rviz.launch.py for centralized RViz configuration.
- Created multi_robot.rviz and single_robot.rviz for visualizing multiple robots.
- Modified ur.urdf.xacro to support multi-robot naming conventions.

File: src/02_robot_startup/urdf/ur.urdf.xacro (robot description, xacro)
@@ -49,10 +49,10 @@
   <!-- convert to property to use substitution in function -->
   <xacro:property name="initial_positions_file" default="$(arg initial_positions_file)"/>
-  <!-- create link fixed to the "world" -->
-  <link name="world" />
+  <!-- create link fixed to the "world" with tf_prefix for multi-robot support -->
+  <link name="$(arg tf_prefix)world" />
   <xacro:ur_robot
     name="$(arg name)"
     tf_prefix="$(arg tf_prefix)"
-    parent="world"
+    parent="$(arg tf_prefix)world"
     joint_limits_parameters_file="$(arg joint_limit_params)"
     kinematics_parameters_file="$(arg kinematics_params)"

Commit message: Refactor launch files and RViz configurations for multi-robot support

File: src/02_robot_startup/urdf/ur.urdf.xacro (robot description, xacro)
@@ -49,5 +49,5 @@
   <!-- convert to property to use substitution in function -->
   <xacro:property name="initial_positions_file" default="$(arg initial_positions_file)"/>
-  <!-- create link fixed to the "world" with tf_prefix for multi-robot support -->
+  <!-- Create robot-specific world link with tf_prefix for multi-robot support -->
   <link name="$(arg tf_prefix)world" />
   <xacro:ur_robot
@@ -63,5 +63,5 @@
     safety_k_position="$(arg safety_k_position)"
     >
-     <origin xyz="0 0 0" rpy="0 0 0" />          <!-- position robot in the world -->
+     <origin xyz="0 0 0" rpy="0 0 0" />
   </xacro:ur_robot>
   <!-- ros2 control instance -->
