Commit message: commit

File: src/rsy_robot_startup/config/ur.urdf.xacro (robot description, xacro)
@@ -76,4 +76,25 @@
   <!-- create link fixed to the "world" -->
   <link name="world" />
+<link name="ground_plane">
+  <collision>
+    <geometry>
+      <box size="3.0 3.0 0.01"/>
+    </geometry>
+    <origin xyz="-0.385 -0.3275 -0.005" rpy="0 0 0"/>
+  </collision>
+  <visual>
+    <geometry>
+      <box size="3.0 3.0 0.01"/>
+    </geometry>
+    <origin xyz="-0.385 -0.3275 -0.005" rpy="0 0 0"/>
+    <material name="yellow">
+      <color rgba="1.0 1.0 0.0 1.0"/>
+    </material>
+  </visual>
+</link>
+<joint name="world_to_ground" type="fixed">
+  <parent link="world"/>
+  <child link="ground_plane"/>
+</joint>
 <xacro:ur_robot
     name="robot1"
@@ -87,5 +108,5 @@
     safety_pos_margin="$(arg robot1_safety_pos_margin)"
     safety_k_position="$(arg robot1_safety_k_position)">
-     <origin xyz="0 0 0" rpy="0 0 0" />          <!-- position robot in the world -->
+     <origin xyz="-0.77 -0.655 0" rpy="0 0 0" />          <!-- position robot in the world -->
 </xacro:ur_robot>
 <xacro:ur_robot
@@ -100,5 +121,5 @@
     safety_pos_margin="$(arg robot2_safety_pos_margin)"
     safety_k_position="$(arg robot2_safety_k_position)">
-     <origin xyz="0 -1.5 0" rpy="0 0 0" />          <!-- position robot in the world -->
+     <origin xyz="0 0 0" rpy="0 0 0" />          <!-- position robot in the world -->
 </xacro:ur_robot>
 <!-- ros2 control instance -->

Commit message: commit

File: src/rsy_robot_startup/config/ur.urdf.xacro (robot description, xacro)
@@ -96,4 +96,25 @@
   <parent link="world"/>
   <child link="ground_plane"/>
+</joint>
+<link name="coneyor_belt">
+  <collision>
+    <geometry>
+      <box size="0.2 0.8 0.1"/>
+    </geometry>
+    <origin xyz="-0.3275 -0.385 0.05" rpy="0 0 0"/>
+  </collision>
+  <visual>
+    <geometry>
+      <box size="0.2 0.8 0.1"/>
+    </geometry>
+    <origin xyz="-0.3275 -0.385 0.05" rpy="0 0 0"/>
+    <material name="yellow">
+      <color rgba="1.0 1.0 0.0 1.0"/>
+    </material>
+  </visual>
+</link>
+<joint name="world_to_coneyor_belt" type="fixed">
+  <parent link="world"/>
+  <child link="coneyor_belt"/>
 </joint>
 <xacro:ur_robot

Commit message: Fix conveyor belt dimensions and adjust robot positions in URDF configuration

File: src/rsy_robot_startup/config/ur.urdf.xacro (robot description, xacro)
@@ -100,13 +100,13 @@
   <collision>
     <geometry>
-      <box size="0.2 0.8 0.1"/>
-    </geometry>
-    <origin xyz="-0.3275 -0.385 0.05" rpy="0 0 0"/>
+      <box size="0.8 0.2 0.1"/>
+    </geometry>
+    <origin xyz="-0.385 0.3275 0.05" rpy="0 0 0"/>
   </collision>
   <visual>
     <geometry>
-      <box size="0.2 0.8 0.1"/>
-    </geometry>
-    <origin xyz="-0.3275 -0.385 0.05" rpy="0 0 0"/>
+      <box size="0.8 0.2 0.1"/>
+    </geometry>
+    <origin xyz="-0.385 0.3275 0.05" rpy="0 0 0"/>
     <material name="yellow">
       <color rgba="1.0 1.0 0.0 1.0"/>
@@ -129,5 +129,5 @@
     safety_pos_margin="$(arg robot1_safety_pos_margin)"
     safety_k_position="$(arg robot1_safety_k_position)">
-     <origin xyz="-0.77 -0.655 0" rpy="0 0 0" />          <!-- position robot in the world -->
+     <origin xyz="0 0 0" rpy="0 0 0" />          <!-- position robot in the world -->
 </xacro:ur_robot>
 <xacro:ur_robot
@@ -142,5 +142,5 @@
     safety_pos_margin="$(arg robot2_safety_pos_margin)"
     safety_k_position="$(arg robot2_safety_k_position)">
-     <origin xyz="0 0 0" rpy="0 0 0" />          <!-- position robot in the world -->
+     <origin xyz="-0.77 0.655 0" rpy="0 0 0" />          <!-- position robot in the world -->
 </xacro:ur_robot>
 <!-- ros2 control instance -->

Commit message: Fix ground plane dimensions and adjust origin in URDF configuration

File: src/rsy_robot_startup/config/ur.urdf.xacro (robot description, xacro)
@@ -79,13 +79,13 @@
   <collision>
     <geometry>
-      <box size="3.0 3.0 0.01"/>
-    </geometry>
-    <origin xyz="-0.385 -0.3275 -0.005" rpy="0 0 0"/>
+      <box size="1.5 1.5 0.01"/>
+    </geometry>
+    <origin xyz="-0.385 0.3275 -0.005" rpy="0 0 0"/>
   </collision>
   <visual>
     <geometry>
-      <box size="3.0 3.0 0.01"/>
-    </geometry>
-    <origin xyz="-0.385 -0.3275 -0.005" rpy="0 0 0"/>
+      <box size="1.5 1.5 0.01"/>
+    </geometry>
+    <origin xyz="-0.385 0.3275 -0.005" rpy="0 0 0"/>
     <material name="yellow">
       <color rgba="1.0 1.0 0.0 1.0"/>

Commit message: Update cube poses and kinematics configuration for improved accuracy and performance

File: src/rsy_robot_startup/config/ur.urdf.xacro (robot description, xacro)
@@ -102,5 +102,5 @@
       <box size="0.8 0.2 0.1"/>
     </geometry>
-    <origin xyz="-0.385 0.3275 0.05" rpy="0 0 0"/>
+    <origin xyz="-0.385 0.3275 -0.05" rpy="0 0 0"/>
   </collision>
   <visual>
@@ -108,5 +108,5 @@
       <box size="0.8 0.2 0.1"/>
     </geometry>
-    <origin xyz="-0.385 0.3275 0.05" rpy="0 0 0"/>
+    <origin xyz="-0.385 0.3275 -0.05" rpy="0 0 0"/>
     <material name="yellow">
       <color rgba="1.0 1.0 0.0 1.0"/>

Commit message: Enhance robot configuration: add TRAC-IK plugin, refine joint limits, and update kinematics settings for improved performance

File: src/rsy_robot_startup/config/ur.urdf.xacro (robot description, xacro)
@@ -102,5 +102,5 @@
       <box size="0.8 0.2 0.1"/>
     </geometry>
-    <origin xyz="-0.385 0.3275 -0.05" rpy="0 0 0"/>
+    <origin xyz="-0.385 0.3275 0.05" rpy="0 0 0"/>
   </collision>
   <visual>
@@ -108,5 +108,5 @@
       <box size="0.8 0.2 0.1"/>
     </geometry>
-    <origin xyz="-0.385 0.3275 -0.05" rpy="0 0 0"/>
+    <origin xyz="-0.385 0.3275 0.05" rpy="0 0 0"/>
     <material name="yellow">
       <color rgba="1.0 1.0 0.0 1.0"/>

Commit message: commikt

File: src/rsy_robot_startup/config/ur.urdf.xacro (robot description, xacro)
@@ -5,4 +5,5 @@
   <xacro:include filename="$(find ur_robot_driver)/urdf/ur.ros2_control.xacro" />
   <xacro:include filename="$(find ur_description)/urdf/inc/ur_transmissions.xacro" />
+  <xacro:include filename="$(find robotiq_description)/urdf/robotiq_2f_85_macro.urdf.xacro" />
   <!-- possible 'ur_type' values: ur3, ur3e, ur5, ur5e, ur7e, ur10, ur10e, ur12e, ur16e, ur8long, ur15, ur18, ur20, ur30 -->
   <!-- the default value should raise an error in case this was called without defining the type -->
@@ -102,5 +103,5 @@
       <box size="0.8 0.2 0.1"/>
     </geometry>
-    <origin xyz="-0.385 0.3275 0.05" rpy="0 0 0"/>
+    <origin xyz="-0.385 0.3275 -0.05" rpy="0 0 0"/>
   </collision>
   <visual>
@@ -108,5 +109,5 @@
       <box size="0.8 0.2 0.1"/>
     </geometry>
-    <origin xyz="-0.385 0.3275 0.05" rpy="0 0 0"/>
+    <origin xyz="-0.385 0.3275 -0.05" rpy="0 0 0"/>
     <material name="yellow">
       <color rgba="1.0 1.0 0.0 1.0"/>

Commit message: commit

File: src/rsy_robot_startup/config/ur.urdf.xacro (robot description, xacro)
@@ -5,21 +5,20 @@
   <xacro:include filename="$(find ur_robot_driver)/urdf/ur.ros2_control.xacro" />
   <xacro:include filename="$(find ur_description)/urdf/inc/ur_transmissions.xacro" />
-  <xacro:include filename="$(find robotiq_description)/urdf/robotiq_2f_85_macro.urdf.xacro" />
-  <!-- possible 'ur_type' values: ur3, ur3e, ur5, ur5e, ur7e, ur10, ur10e, ur12e, ur16e, ur8long, ur15, ur18, ur20, ur30 -->
-  <!-- the default value should raise an error in case this was called without defining the type -->
+  <!-- Robot 1: UR3 configuration -->
   <xacro:arg name="robot1_ur_type" default="ur3"/>
-  <xacro:arg name="robot1_joint_limit_params" default="$(find ur_description)/config/$(arg robot1_ur_type)/joint_limits.yaml"/>
-  <xacro:arg name="robot1_kinematics_params" default="$(find ur_description)/config/$(arg robot1_ur_type)/default_kinematics.yaml"/>
-  <xacro:arg name="robot1_physical_params" default="$(find ur_description)/config/$(arg robot1_ur_type)/physical_parameters.yaml"/>
-  <xacro:arg name="robot1_visual_params" default="$(find ur_description)/config/$(arg robot1_ur_type)/visual_parameters.yaml"/>
+  <xacro:arg name="robot1_joint_limit_params" default="$(find rsy_robot_startup)/config/urdf_joint_limits.yaml"/>
+  <xacro:arg name="robot1_kinematics_params" default="$(find ur_description)/config/ur3/default_kinematics.yaml"/>
+  <xacro:arg name="robot1_physical_params" default="$(find ur_description)/config/ur3/physical_parameters.yaml"/>
+  <xacro:arg name="robot1_visual_params" default="$(find ur_description)/config/ur3/visual_parameters.yaml"/>
   <xacro:arg name="robot1_transmission_hw_interface" default=""/>
   <xacro:arg name="robot1_safety_limits" default="false"/>
   <xacro:arg name="robot1_safety_pos_margin" default="0.15"/>
   <xacro:arg name="robot1_safety_k_position" default="20"/>
+  <!-- Robot 2: UR3e configuration -->
   <xacro:arg name="robot2_ur_type" default="ur3e"/>
-  <xacro:arg name="robot2_joint_limit_params" default="$(find ur_description)/config/$(arg robot2_ur_type)/joint_limits.yaml"/>
-  <xacro:arg name="robot2_kinematics_params" default="$(find ur_description)/config/$(arg robot2_ur_type)/default_kinematics.yaml"/>
-  <xacro:arg name="robot2_physical_params" default="$(find ur_description)/config/$(arg robot2_ur_type)/physical_parameters.yaml"/>
-  <xacro:arg name="robot2_visual_params" default="$(find ur_description)/config/$(arg robot2_ur_type)/visual_parameters.yaml"/>
+  <xacro:arg name="robot2_joint_limit_params" default="$(find rsy_robot_startup)/config/urdf_joint_limits.yaml"/>
+  <xacro:arg name="robot2_kinematics_params" default="$(find ur_description)/config/ur3e/default_kinematics.yaml"/>
+  <xacro:arg name="robot2_physical_params" default="$(find ur_description)/config/ur3e/physical_parameters.yaml"/>
+  <xacro:arg name="robot2_visual_params" default="$(find ur_description)/config/ur3e/visual_parameters.yaml"/>
   <xacro:arg name="robot2_transmission_hw_interface" default=""/>
   <xacro:arg name="robot2_safety_limits" default="false"/>
@@ -103,5 +102,5 @@
       <box size="0.8 0.2 0.1"/>
     </geometry>
-    <origin xyz="-0.385 0.3275 -0.05" rpy="0 0 0"/>
+    <origin xyz="-0.385 0.3275 0.05" rpy="0 0 0"/>
   </collision>
   <visual>
@@ -109,5 +108,5 @@
       <box size="0.8 0.2 0.1"/>
     </geometry>
-    <origin xyz="-0.385 0.3275 -0.05" rpy="0 0 0"/>
+    <origin xyz="-0.385 0.3275 0.05" rpy="0 0 0"/>
     <material name="yellow">
       <color rgba="1.0 1.0 0.0 1.0"/>

Commit message: commit

File: src/rsy_robot_startup/config/ur.urdf.xacro (robot description, xacro)
@@ -27,9 +27,9 @@
 <!-- ros2_control related parameters for robot1 -->
 <xacro:arg name="robot1_headless_mode" default="false" />
-<xacro:arg name="robot1_robot_ip" default="0.0.0.0" />
+<xacro:arg name="robot1_robot_ip" default="192.168.0.51" />
 <xacro:arg name="robot1_script_filename" default=""/>
 <xacro:arg name="robot1_output_recipe_filename" default=""/>
 <xacro:arg name="robot1_input_recipe_filename" default=""/>
-<xacro:arg name="robot1_reverse_ip" default="0.0.0.0"/>
+<xacro:arg name="robot1_reverse_ip" default="192.168.0.2"/>
 <xacro:arg name="robot1_script_command_port" default="50004"/>
 <xacro:arg name="robot1_reverse_port" default="50001"/>
@@ -48,9 +48,9 @@
 <!-- ros2_control related parameters for robot2 -->
 <xacro:arg name="robot2_headless_mode" default="false" />
-<xacro:arg name="robot2_robot_ip" default="0.0.0.0" />
+<xacro:arg name="robot2_robot_ip" default="192.168.0.11" />
 <xacro:arg name="robot2_script_filename" default=""/>
 <xacro:arg name="robot2_output_recipe_filename" default=""/>
 <xacro:arg name="robot2_input_recipe_filename" default=""/>
-<xacro:arg name="robot2_reverse_ip" default="0.0.0.0"/>
+<xacro:arg name="robot2_reverse_ip" default="192.168.0.2"/>
 <xacro:arg name="robot2_script_command_port" default="50014"/>
 <xacro:arg name="robot2_reverse_port" default="50011"/>
@@ -68,5 +68,5 @@
 <xacro:arg name="robot2_tool_tcp_port" default="54322" />
     <!-- Simulation parameters -->
-  <xacro:arg name="use_mock_hardware" default="true" />
+  <xacro:arg name="use_mock_hardware" default="false" />
   <xacro:arg name="mock_sensor_commands" default="false" />
   <!-- initial position for simulations (Mock Hardware, Gazebo, Ignition) -->
@@ -129,5 +129,5 @@
     safety_pos_margin="$(arg robot1_safety_pos_margin)"
     safety_k_position="$(arg robot1_safety_k_position)">
-     <origin xyz="0 0 0" rpy="0 0 0" />          <!-- position robot in the world -->
+     <origin xyz="0.77 -0.655 0" rpy="0 0 1.570796" />          <!-- position robot in the world -->
 </xacro:ur_robot>
 <xacro:ur_robot
@@ -142,5 +142,5 @@
     safety_pos_margin="$(arg robot2_safety_pos_margin)"
     safety_k_position="$(arg robot2_safety_k_position)">
-     <origin xyz="-0.77 0.655 0" rpy="0 0 0" />          <!-- position robot in the world -->
+     <origin xyz="0 0 0" rpy="0 0 0" />          <!-- position robot in the world -->
 </xacro:ur_robot>
 <!-- ros2 control instance -->

Commit message: Add static Robotiq gripper configuration and update URDF files

File: src/rsy_robot_startup/config/ur.urdf.xacro (robot description, xacro)
@@ -5,4 +5,6 @@
   <xacro:include filename="$(find ur_robot_driver)/urdf/ur.ros2_control.xacro" />
   <xacro:include filename="$(find ur_description)/urdf/inc/ur_transmissions.xacro" />
+  <!-- Static Robotiq gripper (visual only) -->
+  <xacro:include filename="$(find rsy_robot_startup)/config/robotiq_2f_85_static.xacro" />
   <!-- Robot 1: UR3 configuration -->
   <xacro:arg name="robot1_ur_type" default="ur3"/>
@@ -68,5 +70,5 @@
 <xacro:arg name="robot2_tool_tcp_port" default="54322" />
     <!-- Simulation parameters -->
-  <xacro:arg name="use_mock_hardware" default="false" />
+  <xacro:arg name="use_mock_hardware" default="true" />
   <xacro:arg name="mock_sensor_commands" default="false" />
   <!-- initial position for simulations (Mock Hardware, Gazebo, Ignition) -->
@@ -144,4 +146,11 @@
      <origin xyz="0 0 0" rpy="0 0 0" />          <!-- position robot in the world -->
 </xacro:ur_robot>
+<!-- Static Robotiq grippers attached to robot tool0 links -->
+<xacro:robotiq_gripper_static prefix="robot1_" parent="robot1_tool0">
+    <origin xyz="0 0 0" rpy="0 0 0" />
+</xacro:robotiq_gripper_static>
+<xacro:robotiq_gripper_static prefix="robot2_" parent="robot2_tool0">
+    <origin xyz="0 0 0" rpy="0 0 0" />
+</xacro:robotiq_gripper_static>
 <!-- ros2 control instance -->
 <xacro:ur_ros2_control

Commit message: Update MoveIt configurations to use TCP links for both robots and adjust RViz display settings

File: src/rsy_robot_startup/config/ur.urdf.xacro (robot description, xacro)
@@ -153,4 +153,17 @@
     <origin xyz="0 0 0" rpy="0 0 0" />
 </xacro:robotiq_gripper_static>
+<!-- TCP (Tool Center Point) links - 16.5cm from tool0 in z direction -->
+<link name="robot1_tcp" />
+<joint name="robot1_tool0_to_tcp" type="fixed">
+    <parent link="robot1_tool0" />
+    <child link="robot1_tcp" />
+    <origin xyz="0 0 0.165" rpy="0 0 0" />
+</joint>
+<link name="robot2_tcp" />
+<joint name="robot2_tool0_to_tcp" type="fixed">
+    <parent link="robot2_tool0" />
+    <child link="robot2_tcp" />
+    <origin xyz="0 0 0.165" rpy="0 0 0" />
+</joint>
 <!-- ros2 control instance -->
 <xacro:ur_ros2_control

Commit message: Update URDF and SRDF configurations for robot gripper self-collisions and adjust robot positions

File: src/rsy_robot_startup/config/ur.urdf.xacro (robot description, xacro)
@@ -131,5 +131,5 @@
     safety_pos_margin="$(arg robot1_safety_pos_margin)"
     safety_k_position="$(arg robot1_safety_k_position)">
-     <origin xyz="0.77 -0.655 0" rpy="0 0 1.570796" />          <!-- position robot in the world -->
+     <origin xyz="0 0 0" rpy="0 0 1.570796" />          <!-- position robot in the world -->
 </xacro:ur_robot>
 <xacro:ur_robot
@@ -144,5 +144,5 @@
     safety_pos_margin="$(arg robot2_safety_pos_margin)"
     safety_k_position="$(arg robot2_safety_k_position)">
-     <origin xyz="0 0 0" rpy="0 0 0" />          <!-- position robot in the world -->
+     <origin xyz="-0.77 0.655 0" rpy="0 0 3.141592" />          <!-- position robot in the world -->
 </xacro:ur_robot>
 <!-- Static Robotiq grippers attached to robot tool0 links -->

Commit message: commit

File: src/rsy_robot_startup/config/ur.urdf.xacro (robot description, xacro)
@@ -120,4 +120,50 @@
   <child link="coneyor_belt"/>
 </joint>
+<!-- ITEM Profile 1 -->
+<link name="item_profile_1">
+  <collision>
+    <geometry>
+      <box size="0.04 0.04 1.0"/>
+    </geometry>
+    <origin xyz="0 0 0.5" rpy="0 0 0"/>
+  </collision>
+  <visual>
+    <geometry>
+      <box size="0.04 0.04 1.0"/>
+    </geometry>
+    <origin xyz="0 0 0.5" rpy="0 0 0"/>
+    <material name="yellow">
+      <color rgba="1.0 1.0 0.0 1.0"/>
+    </material>
+  </visual>
+</link>
+<joint name="world_to_item_profile_1" type="fixed">
+  <parent link="world"/>
+  <child link="item_profile_1"/>
+  <origin xyz="0.30 -0.30 0" rpy="0 0 0"/>
+</joint>
+<!-- ITEM Profile 2 -->
+<link name="item_profile_2">
+  <collision>
+    <geometry>
+      <box size="0.04 0.04 1.0"/>
+    </geometry>
+    <origin xyz="0 0 0.5" rpy="0 0 0"/>
+  </collision>
+  <visual>
+    <geometry>
+      <box size="0.04 0.04 1.0"/>
+    </geometry>
+    <origin xyz="0 0 0.5" rpy="0 0 0"/>
+    <material name="yellow">
+      <color rgba="1.0 1.0 0.0 1.0"/>
+    </material>
+  </visual>
+</link>
+<joint name="world_to_item_profile_2" type="fixed">
+  <parent link="world"/>
+  <child link="item_profile_2"/>
+  <origin xyz="-1.07 0.955 0" rpy="0 0 0"/>
+</joint>
 <xacro:ur_robot
     name="robot1"

Commit message: Added global configuration

File: src/rsy_robot_startup/config/ur.urdf.xacro (robot description, xacro)
@@ -69,4 +69,11 @@
 <xacro:arg name="robot2_tool_device_name" default="/tmp/ttyUR2" />
 <xacro:arg name="robot2_tool_tcp_port" default="54322" />
+<!-- Robot2 position relative to world frame -->
+<xacro:arg name="robot2_x" default="-0.77" />
+<xacro:arg name="robot2_y" default="0.655" />
+<xacro:arg name="robot2_z" default="0" />
+<xacro:arg name="robot2_roll" default="0" />
+<xacro:arg name="robot2_pitch" default="0" />
+<xacro:arg name="robot2_yaw" default="3.141592" />
     <!-- Simulation parameters -->
   <xacro:arg name="use_mock_hardware" default="true" />
@@ -144,5 +151,5 @@
     safety_pos_margin="$(arg robot2_safety_pos_margin)"
     safety_k_position="$(arg robot2_safety_k_position)">
-     <origin xyz="-0.77 0.655 0" rpy="0 0 3.141592" />          <!-- position robot in the world -->
+     <origin xyz="$(arg robot2_x) $(arg robot2_y) $(arg robot2_z)" rpy="$(arg robot2_roll) $(arg robot2_pitch) $(arg robot2_yaw)" />
 </xacro:ur_robot>
 <!-- Static Robotiq grippers attached to robot tool0 links -->

Commit message: Abort solving when path planning failed

File: src/rsy_robot_startup/config/ur.urdf.xacro (robot description, xacro)
@@ -104,5 +104,5 @@
       <box size="0.8 0.2 0.1"/>
     </geometry>
-    <origin xyz="-0.385 0.3275 0.05" rpy="0 0 0"/>
+    <origin xyz="-0.385 0.3275 -0.05" rpy="0 0 0"/>
   </collision>
   <visual>
@@ -110,5 +110,5 @@
       <box size="0.8 0.2 0.1"/>
     </geometry>
-    <origin xyz="-0.385 0.3275 0.05" rpy="0 0 0"/>
+    <origin xyz="-0.385 0.3275 -0.05" rpy="0 0 0"/>
     <material name="yellow">
       <color rgba="1.0 1.0 0.0 1.0"/>
