Commit message: Update system configuration and resource files for robot1 and robot2
- Disable mock hardware usage for robot1 and enable for robot2
- Update gripper IP addresses to match the robot IPs
- Increase joint velocity limits for robot1 and robot2
- Adjust translational velocity limits for the Pilz planner
- Add RTDE input and output recipe files for robot1 and robot2
- Modify launch file to handle new mock hardware arguments and URScript interfaces

File: src/rsy_robot_startup/config/ur.urdf.xacro (robot description, xacro)
@@ -10,5 +10,5 @@
   <xacro:arg name="robot1_ur_type" default="ur3"/>
   <xacro:arg name="robot1_joint_limit_params" default="$(find rsy_robot_startup)/config/urdf_joint_limits.yaml"/>
-  <xacro:arg name="robot1_kinematics_params" default="$(find ur_description)/config/ur3/default_kinematics.yaml"/>
+  <xacro:arg name="robot1_kinematics_params" default="$(find rsy_robot_startup)/config/ur3_calibration.yaml"/>
   <xacro:arg name="robot1_physical_params" default="$(find ur_description)/config/ur3/physical_parameters.yaml"/>
   <xacro:arg name="robot1_visual_params" default="$(find ur_description)/config/ur3/visual_parameters.yaml"/>
@@ -20,5 +20,5 @@
   <xacro:arg name="robot2_ur_type" default="ur3e"/>
   <xacro:arg name="robot2_joint_limit_params" default="$(find rsy_robot_startup)/config/urdf_joint_limits.yaml"/>
-  <xacro:arg name="robot2_kinematics_params" default="$(find ur_description)/config/ur3e/default_kinematics.yaml"/>
+  <xacro:arg name="robot2_kinematics_params" default="$(find rsy_robot_startup)/config/ur3e_calibration.yaml"/>
   <xacro:arg name="robot2_physical_params" default="$(find ur_description)/config/ur3e/physical_parameters.yaml"/>
   <xacro:arg name="robot2_visual_params" default="$(find ur_description)/config/ur3e/visual_parameters.yaml"/>
@@ -30,8 +30,8 @@
 <xacro:arg name="robot1_headless_mode" default="false" />
 <xacro:arg name="robot1_robot_ip" default="192.168.0.51" />
-<xacro:arg name="robot1_script_filename" default=""/>
-<xacro:arg name="robot1_output_recipe_filename" default=""/>
-<xacro:arg name="robot1_input_recipe_filename" default=""/>
-<xacro:arg name="robot1_reverse_ip" default="192.168.0.2"/>
+<xacro:arg name="robot1_script_filename" default="$(find ur_client_library)/resources/external_control.urscript"/>
+<xacro:arg name="robot1_output_recipe_filename" default="$(find rsy_robot_startup)/resources/robot1_rtde_output_recipe.txt"/>
+<xacro:arg name="robot1_input_recipe_filename" default="$(find rsy_robot_startup)/resources/robot1_rtde_input_recipe.txt"/>
+<xacro:arg name="robot1_reverse_ip" default="192.168.0.100"/>
 <xacro:arg name="robot1_script_command_port" default="50004"/>
 <xacro:arg name="robot1_reverse_port" default="50001"/>
@@ -51,8 +51,8 @@
 <xacro:arg name="robot2_headless_mode" default="false" />
 <xacro:arg name="robot2_robot_ip" default="192.168.0.11" />
-<xacro:arg name="robot2_script_filename" default=""/>
-<xacro:arg name="robot2_output_recipe_filename" default=""/>
-<xacro:arg name="robot2_input_recipe_filename" default=""/>
-<xacro:arg name="robot2_reverse_ip" default="192.168.0.2"/>
+<xacro:arg name="robot2_script_filename" default="$(find ur_client_library)/resources/external_control.urscript"/>
+<xacro:arg name="robot2_output_recipe_filename" default="$(find rsy_robot_startup)/resources/robot2_rtde_output_recipe.txt"/>
+<xacro:arg name="robot2_input_recipe_filename" default="$(find rsy_robot_startup)/resources/robot2_rtde_input_recipe.txt"/>
+<xacro:arg name="robot2_reverse_ip" default="192.168.0.100"/>
 <xacro:arg name="robot2_script_command_port" default="50014"/>
 <xacro:arg name="robot2_reverse_port" default="50011"/>
@@ -77,5 +77,6 @@
 <xacro:arg name="robot2_yaw" default="3.141592" />
     <!-- Simulation parameters -->
-  <xacro:arg name="use_mock_hardware" default="true" />
+  <xacro:arg name="robot1_use_mock_hardware" default="true" />
+  <xacro:arg name="robot2_use_mock_hardware" default="true" />
   <xacro:arg name="mock_sensor_commands" default="false" />
   <!-- initial position for simulations (Mock Hardware, Gazebo, Ignition) -->
@@ -201,5 +202,5 @@
 <!-- Static Robotiq grippers attached to robot tool0 links -->
 <xacro:robotiq_gripper_static prefix="robot1_" parent="robot1_tool0">
-    <origin xyz="0 0 0" rpy="0 0 0" />
+    <origin xyz="0 0 0" rpy="0 0 1.570796" />
 </xacro:robotiq_gripper_static>
 <xacro:robotiq_gripper_static prefix="robot2_" parent="robot2_tool0">
@@ -224,6 +225,5 @@
     tf_prefix="robot1_"
     kinematics_parameters_file="$(arg robot1_kinematics_params)"
-    transmission_hw_interface="$(arg robot1_transmission_hw_interface)"
-    use_mock_hardware="$(arg use_mock_hardware)"
+    use_mock_hardware="$(arg robot1_use_mock_hardware)"
     mock_sensor_commands="$(arg mock_sensor_commands)"
     headless_mode="$(arg robot1_headless_mode)"
@@ -252,6 +252,5 @@
     tf_prefix="robot2_"
     kinematics_parameters_file="$(arg robot2_kinematics_params)"
-    transmission_hw_interface="$(arg robot2_transmission_hw_interface)"
-    use_mock_hardware="$(arg use_mock_hardware)"
+    use_mock_hardware="$(arg robot2_use_mock_hardware)"
     mock_sensor_commands="$(arg mock_sensor_commands)"
     headless_mode="$(arg robot2_headless_mode)"

Commit message: Add robot configuration and update launch file for improved hardware integration

File: src/rsy_robot_startup/config/ur.urdf.xacro (robot description, xacro)
@@ -212,5 +212,5 @@
     <parent link="robot1_tool0" />
     <child link="robot1_tcp" />
-    <origin xyz="0 0 0.165" rpy="0 0 0" />
+    <origin xyz="0 0 0.165" rpy="0 0 1.570796" />
 </joint>
 <link name="robot2_tcp" />

Commit message: Update box dimensions for item profiles in URDF configuration

File: src/rsy_robot_startup/config/ur.urdf.xacro (robot description, xacro)
@@ -132,11 +132,11 @@
   <collision>
     <geometry>
-      <box size="0.04 0.04 1.0"/>
-    </geometry>
-    <origin xyz="0 0 0.5" rpy="0 0 0"/>
-  </collision>
-  <visual>
-    <geometry>
-      <box size="0.04 0.04 1.0"/>
+      <box size="0.20 0.20 1.0"/>
+    </geometry>
+    <origin xyz="0 0 0.5" rpy="0 0 0"/>
+  </collision>
+  <visual>
+    <geometry>
+      <box size="0.15 0.15 1.0"/>
     </geometry>
     <origin xyz="0 0 0.5" rpy="0 0 0"/>
@@ -155,11 +155,11 @@
   <collision>
     <geometry>
-      <box size="0.04 0.04 1.0"/>
-    </geometry>
-    <origin xyz="0 0 0.5" rpy="0 0 0"/>
-  </collision>
-  <visual>
-    <geometry>
-      <box size="0.04 0.04 1.0"/>
+      <box size="0.15 0.15 1.0"/>
+    </geometry>
+    <origin xyz="0 0 0.5" rpy="0 0 0"/>
+  </collision>
+  <visual>
+    <geometry>
+      <box size="0.15 0.15 1.0"/>
     </geometry>
     <origin xyz="0 0 0.5" rpy="0 0 0"/>

Commit message: feat: Update cube poses and offsets for improved motion planning accuracy

File: src/rsy_robot_startup/config/ur.urdf.xacro (robot description, xacro)
@@ -174,4 +174,50 @@
   <origin xyz="-1.07 0.955 0" rpy="0 0 0"/>
 </joint>
+<!-- CUBE Robot1 -->
+<link name="cube_robot1">
+  <collision>
+    <geometry>
+      <box size="0.06 0.06 0.06"/>
+    </geometry>
+    <origin xyz="0.03 0.03 0.03" rpy="0 0 0"/>
+  </collision>
+  <visual>
+    <geometry>
+      <box size="0.06 0.06 0.06"/>
+    </geometry>
+    <origin xyz="0.03 0.03 0.03" rpy="0 0 0"/>
+    <material name="yellow">
+      <color rgba="1.0 1.0 0.0 1.0"/>
+    </material>
+  </visual>
+</link>
+<joint name="robot1_tcp_to_cube_robot1" type="fixed">
+  <parent link="robot1_tcp"/>
+  <child link="cube_robot1"/>
+  <origin xyz="-0.03 -0.03 -0.03" rpy="0 0 0"/>
+</joint>
+<!-- CUBE Robot2 -->
+<link name="cube_robot2">
+  <collision>
+    <geometry>
+      <box size="0.06 0.06 0.06"/>
+    </geometry>
+    <origin xyz="0.03 0.03 0.03" rpy="0 0 0"/>
+  </collision>
+  <visual>
+    <geometry>
+      <box size="0.06 0.06 0.06"/>
+    </geometry>
+    <origin xyz="0.03 0.03 0.03" rpy="0 0 0"/>
+    <material name="yellow">
+      <color rgba="1.0 1.0 0.0 1.0"/>
+    </material>
+  </visual>
+</link>
+<joint name="robot2_tcp_to_cube_robot2" type="fixed">
+  <parent link="robot2_tcp"/>
+  <child link="cube_robot2"/>
+  <origin xyz="-0.03 -0.03 -0.03" rpy="0 0 0"/>
+</joint>
 <xacro:ur_robot
     name="robot1"

Commit message: feat: Update robot configurations for improved accuracy and collision handling

File: src/rsy_robot_startup/config/ur.urdf.xacro (robot description, xacro)
@@ -70,6 +70,6 @@
 <xacro:arg name="robot2_tool_tcp_port" default="54322" />
 <!-- Robot2 position relative to world frame -->
-<xacro:arg name="robot2_x" default="-0.77" />
-<xacro:arg name="robot2_y" default="0.655" />
+<xacro:arg name="robot2_x" default="-0.76626" />
+<xacro:arg name="robot2_y" default="0.64864" />
 <xacro:arg name="robot2_z" default="0" />
 <xacro:arg name="robot2_roll" default="0" />
@@ -86,61 +86,144 @@
   <!-- create link fixed to the "world" -->
   <link name="world" />
-<link name="ground_plane">
+  <link name="ground_plane">
+    <collision>
+      <geometry>
+        <box size="2.0 2.0 0.01"/>
+      </geometry>
+      <origin xyz="-0.38313 0.32432 -0.005" rpy="0 0 0"/>
+    </collision>
+    <visual>
+      <geometry>
+        <box size="2.0 2.0 0.01"/>
+      </geometry>
+      <origin xyz="-0.38313 0.32432 -0.005" rpy="0 0 0"/>
+      <material name="yellow">
+        <color rgba="1.0 1.0 0.0 0.1"/>
+      </material>
+    </visual>
+  </link>
+  <joint name="world_to_ground" type="fixed">
+    <parent link="world"/>
+    <child link="ground_plane"/>
+  </joint>
+  <link name="wall_left">
+    <collision>
+      <geometry>
+        <box size="0.01 1.44864 1.0"/>
+      </geometry>
+      <origin xyz="0.405 0.32432 0.5" rpy="0 0 0"/>
+    </collision>
+    <visual>
+      <geometry>
+        <box size="0.01 1.44864 1.0"/>
+      </geometry>
+      <origin xyz="0.405 0.32432 0.5" rpy="0 0 0"/>
+      <material name="yellow">
+        <color rgba="1.0 1.0 0.0 0.1"/>
+      </material>
+    </visual>
+  </link>
+  <joint name="world_to_wall_left" type="fixed">
+    <parent link="world"/>
+    <child link="wall_left"/>
+  </joint>
+  <link name="wall_right">
+    <collision>
+      <geometry>
+        <box size="0.01 1.44864 1.0"/>
+      </geometry>
+      <origin xyz="-1.17126 0.32432 0.5" rpy="0 0 0"/>
+    </collision>
+    <visual>
+      <geometry>
+        <box size="0.01 1.44864 1.0"/>
+      </geometry>
+      <origin xyz="-1.17126 0.32432 0.5" rpy="0 0 0"/>
+      <material name="yellow">
+        <color rgba="1.0 1.0 0.0 0.1"/>
+      </material>
+    </visual>
+  </link>
+  <joint name="world_to_wall_right" type="fixed">
+    <parent link="world"/>
+    <child link="wall_right"/>
+  </joint>
+  <link name="wall_back">
+    <collision>
+      <geometry>
+        <box size="1.56626 0.01 1.0"/>
+      </geometry>
+      <origin xyz="-0.38313 -0.405 0.5" rpy="0 0 0"/>
+    </collision>
+    <visual>
+      <geometry>
+        <box size="1.56626 0.01 1.0"/>
+      </geometry>
+      <origin xyz="-0.38313 -0.405 0.5" rpy="0 0 0"/>
+      <material name="yellow">
+        <color rgba="1.0 1.0 0.0 0.1"/>
+      </material>
+    </visual>
+  </link>
+  <joint name="world_to_wall_back" type="fixed">
+    <parent link="world"/>
+    <child link="wall_back"/>
+  </joint>
+  <link name="wall_front">
+    <collision>
+      <geometry>
+        <box size="1.56626 0.01 1.0"/>
+      </geometry>
+      <origin xyz="-0.38313 1.05364 0.5" rpy="0 0 0"/>
+    </collision>
+    <visual>
+      <geometry>
+        <box size="1.56626 0.01 1.0"/>
+      </geometry>
+      <origin xyz="-0.38313 1.05364 0.5" rpy="0 0 0"/>
+      <material name="yellow">
+        <color rgba="1.0 1.0 0.0 0.1"/>
+      </material>
+    </visual>
+  </link>
+  <joint name="world_to_wall_front" type="fixed">
+    <parent link="world"/>
+    <child link="wall_front"/>
+  </joint>
+  <link name="roof">
+    <collision>
+      <geometry>
+        <box size="2.0 2.0 0.01"/>
+      </geometry>
+      <origin xyz="-0.38313 0.32432 1.005" rpy="0 0 0"/>
+    </collision>
+    <visual>
+      <geometry>
+        <box size="2.0 2.0 0.01"/>
+      </geometry>
+      <origin xyz="-0.38313 0.32432 1.005" rpy="0 0 0"/>
+      <material name="yellow">
+        <color rgba="1.0 1.0 0.0 0.1"/>
+      </material>
+    </visual>
+  </link>
+  <joint name="world_to_roof" type="fixed">
+    <parent link="world"/>
+    <child link="roof"/>
+  </joint>
+<link name="item_profile_1">
   <collision>
     <geometry>
-      <box size="1.5 1.5 0.01"/>
-    </geometry>
-    <origin xyz="-0.385 0.3275 -0.005" rpy="0 0 0"/>
+      <box size="0.20 0.20 1.0"/>
+    </geometry>
+  <origin xyz="0.30 -0.30 0.5" rpy="0 0 0"/>
   </collision>
   <visual>
     <geometry>
-      <box size="1.5 1.5 0.01"/>
-    </geometry>
-    <origin xyz="-0.385 0.3275 -0.005" rpy="0 0 0"/>
+      <box size="0.20 0.20 1.0"/>
+    </geometry>
+    <origin xyz="0.30 -0.30 0.5" rpy="0 0 0"/>
     <material name="yellow">
-      <color rgba="1.0 1.0 0.0 1.0"/>
-    </material>
-  </visual>
-</link>
-<joint name="world_to_ground" type="fixed">
-  <parent link="world"/>
-  <child link="ground_plane"/>
-</joint>
-<link name="coneyor_belt">
-  <collision>
-    <geometry>
-      <box size="0.8 0.2 0.1"/>
-    </geometry>
-    <origin xyz="-0.385 0.3275 -0.05" rpy="0 0 0"/>
-  </collision>
-  <visual>
-    <geometry>
-      <box size="0.8 0.2 0.1"/>
-    </geometry>
-    <origin xyz="-0.385 0.3275 -0.05" rpy="0 0 0"/>
-    <material name="yellow">
-      <color rgba="1.0 1.0 0.0 1.0"/>
-    </material>
-  </visual>
-</link>
-<joint name="world_to_coneyor_belt" type="fixed">
-  <parent link="world"/>
-  <child link="coneyor_belt"/>
-</joint>
-<!-- ITEM Profile 1 -->
-<link name="item_profile_1">
-  <collision>
-    <geometry>
-      <box size="0.20 0.20 1.0"/>
-    </geometry>
-    <origin xyz="0 0 0.5" rpy="0 0 0"/>
-  </collision>
-  <visual>
-    <geometry>
-      <box size="0.15 0.15 1.0"/>
-    </geometry>
-    <origin xyz="0 0 0.5" rpy="0 0 0"/>
-    <material name="yellow">
-      <color rgba="1.0 1.0 0.0 1.0"/>
+      <color rgba="1.0 1.0 0.0 0.1"/>
     </material>
   </visual>
@@ -149,21 +232,19 @@
   <parent link="world"/>
   <child link="item_profile_1"/>
-  <origin xyz="0.30 -0.30 0" rpy="0 0 0"/>
-</joint>
-<!-- ITEM Profile 2 -->
+</joint>
 <link name="item_profile_2">
   <collision>
     <geometry>
-      <box size="0.15 0.15 1.0"/>
-    </geometry>
-    <origin xyz="0 0 0.5" rpy="0 0 0"/>
+      <box size="0.20 0.20 1.0"/>
+    </geometry>
+    <origin xyz="-1.06626 0.94864 0.5" rpy="0 0 0"/>
   </collision>
   <visual>
     <geometry>
-      <box size="0.15 0.15 1.0"/>
-    </geometry>
-    <origin xyz="0 0 0.5" rpy="0 0 0"/>
+      <box size="0.20 0.20 1.0"/>
+    </geometry>
+    <origin xyz="-1.06626 0.94864 0.5" rpy="0 0 0"/>
     <material name="yellow">
-      <color rgba="1.0 1.0 0.0 1.0"/>
+      <color rgba="1.0 1.0 0.0 0.1"/>
     </material>
   </visual>
@@ -172,7 +253,5 @@
   <parent link="world"/>
   <child link="item_profile_2"/>
-  <origin xyz="-1.07 0.955 0" rpy="0 0 0"/>
-</joint>
-<!-- CUBE Robot1 -->
+</joint>
 <link name="cube_robot1">
   <collision>
@@ -188,5 +267,5 @@
     <origin xyz="0.03 0.03 0.03" rpy="0 0 0"/>
     <material name="yellow">
-      <color rgba="1.0 1.0 0.0 1.0"/>
+      <color rgba="1.0 1.0 0.0 0.1"/>
     </material>
   </visual>
@@ -197,5 +276,4 @@
   <origin xyz="-0.03 -0.03 -0.03" rpy="0 0 0"/>
 </joint>
-<!-- CUBE Robot2 -->
 <link name="cube_robot2">
   <collision>
@@ -211,5 +289,5 @@
     <origin xyz="0.03 0.03 0.03" rpy="0 0 0"/>
     <material name="yellow">
-      <color rgba="1.0 1.0 0.0 1.0"/>
+      <color rgba="1.0 1.0 0.0 0.1"/>
     </material>
   </visual>
@@ -231,5 +309,5 @@
     safety_pos_margin="$(arg robot1_safety_pos_margin)"
     safety_k_position="$(arg robot1_safety_k_position)">
-     <origin xyz="0 0 0" rpy="0 0 1.570796" />          <!-- position robot in the world -->
+     <origin xyz="0 0 0" rpy="0 0 1.570796" />
 </xacro:ur_robot>
 <xacro:ur_robot

Commit message: feat: Update offsets for cube handling and adjust robot joint origins for improved accuracy

File: src/rsy_robot_startup/config/ur.urdf.xacro (robot description, xacro)
@@ -336,5 +336,5 @@
     <parent link="robot1_tool0" />
     <child link="robot1_tcp" />
-    <origin xyz="0 0 0.165" rpy="0 0 1.570796" />
+    <origin xyz="0 0 0.2078" rpy="0 0 1.570796" />
 </joint>
 <link name="robot2_tcp" />
@@ -342,5 +342,5 @@
     <parent link="robot2_tool0" />
     <child link="robot2_tcp" />
-    <origin xyz="0 0 0.165" rpy="0 0 0" />
+    <origin xyz="0 0 0.2078" rpy="0 0 0" />
 </joint>
 <!-- ros2 control instance -->

Commit message: feat: Update mock hardware configurations and enhance cube perception services

File: src/rsy_robot_startup/config/ur.urdf.xacro (robot description, xacro)
@@ -259,5 +259,5 @@
       <box size="0.06 0.06 0.06"/>
     </geometry>
-    <origin xyz="0.03 0.03 0.03" rpy="0 0 0"/>
+    <origin xyz="0.0 0.0 -0.04" rpy="0 0 0"/>
   </collision>
   <visual>
@@ -265,5 +265,5 @@
       <box size="0.06 0.06 0.06"/>
     </geometry>
-    <origin xyz="0.03 0.03 0.03" rpy="0 0 0"/>
+    <origin xyz="0.0 0.0 -0.04" rpy="0 0 0"/>
     <material name="yellow">
       <color rgba="1.0 1.0 0.0 0.1"/>
@@ -274,5 +274,4 @@
   <parent link="robot1_tcp"/>
   <child link="cube_robot1"/>
-  <origin xyz="-0.03 -0.03 -0.03" rpy="0 0 0"/>
 </joint>
 <link name="cube_robot2">
@@ -281,5 +280,5 @@
       <box size="0.06 0.06 0.06"/>
     </geometry>
-    <origin xyz="0.03 0.03 0.03" rpy="0 0 0"/>
+    <origin xyz="0.0 0.0 -0.04" rpy="0 0 0"/>
   </collision>
   <visual>
@@ -287,5 +286,5 @@
       <box size="0.06 0.06 0.06"/>
     </geometry>
-    <origin xyz="0.03 0.03 0.03" rpy="0 0 0"/>
+    <origin xyz="0.0 0.0 -0.04" rpy="0 0 0"/>
     <material name="yellow">
       <color rgba="1.0 1.0 0.0 0.1"/>
@@ -296,5 +295,25 @@
   <parent link="robot2_tcp"/>
   <child link="cube_robot2"/>
-  <origin xyz="-0.03 -0.03 -0.03" rpy="0 0 0"/>
+</joint>
+<link name="cube_stand">
+  <collision>
+    <geometry>
+      <box size="0.07 0.07 0.12"/>
+    </geometry>
+    <origin xyz="-0.15654 0.7294 0.04039" rpy="0 0 0"/>
+  </collision>
+  <visual>
+    <geometry>
+      <box size="0.07 0.07 0.12"/>
+    </geometry>
+    <origin xyz="-0.12654 0.7334 0.04039" rpy="0 0 0"/>
+    <material name="yellow">
+      <color rgba="1.0 1.0 0.0 0.1"/>
+    </material>
+  </visual>
+</link>
+<joint name="world_to_cube_stand" type="fixed">
+  <parent link="world"/>
+  <child link="cube_stand"/>
 </joint>
 <xacro:ur_robot

Commit message: worx

File: src/rsy_robot_startup/config/ur.urdf.xacro (robot description, xacro)
@@ -307,5 +307,5 @@
       <box size="0.07 0.07 0.12"/>
     </geometry>
-    <origin xyz="-0.12654 0.7334 0.04039" rpy="0 0 0"/>
+    <origin xyz="-0.11954 0.7334 0.04039" rpy="0 0 0"/>
     <material name="yellow">
       <color rgba="1.0 1.0 0.0 0.1"/>

Commit message: feat: Update visualization configuration and collision settings for cube robots

File: src/rsy_robot_startup/config/ur.urdf.xacro (robot description, xacro)
@@ -259,11 +259,11 @@
       <box size="0.06 0.06 0.06"/>
     </geometry>
-    <origin xyz="0.0 0.0 -0.04" rpy="0 0 0"/>
-  </collision>
-  <visual>
-    <geometry>
-      <box size="0.06 0.06 0.06"/>
-    </geometry>
-    <origin xyz="0.0 0.0 -0.04" rpy="0 0 0"/>
+    <origin xyz="0.0 0.0 -0.042" rpy="0 0 0"/>
+  </collision>
+  <visual>
+    <geometry>
+      <box size="0.06 0.06 0.06"/>
+    </geometry>
+    <origin xyz="0.0 0.0 -0.042" rpy="0 0 0"/>
     <material name="yellow">
       <color rgba="1.0 1.0 0.0 0.1"/>
@@ -280,11 +280,11 @@
       <box size="0.06 0.06 0.06"/>
     </geometry>
-    <origin xyz="0.0 0.0 -0.04" rpy="0 0 0"/>
-  </collision>
-  <visual>
-    <geometry>
-      <box size="0.06 0.06 0.06"/>
-    </geometry>
-    <origin xyz="0.0 0.0 -0.04" rpy="0 0 0"/>
+    <origin xyz="0.0 0.0 -0.042" rpy="0 0 0"/>
+  </collision>
+  <visual>
+    <geometry>
+      <box size="0.06 0.06 0.06"/>
+    </geometry>
+    <origin xyz="0.0 0.0 -0.042" rpy="0 0 0"/>
     <material name="yellow">
       <color rgba="1.0 1.0 0.0 0.1"/>
@@ -296,16 +296,34 @@
   <child link="cube_robot2"/>
 </joint>
-<link name="cube_stand">
-  <collision>
-    <geometry>
-      <box size="0.07 0.07 0.12"/>
-    </geometry>
-    <origin xyz="-0.15654 0.7294 0.04039" rpy="0 0 0"/>
-  </collision>
-  <visual>
-    <geometry>
-      <box size="0.07 0.07 0.12"/>
-    </geometry>
-    <origin xyz="-0.11954 0.7334 0.04039" rpy="0 0 0"/>
+<link name="cubestand">
+  <collision>
+    <geometry>
+      <mesh filename="package://rsy_robot_startup/meshes/cube_stand.stl" scale="0.001 0.001 0.001"/>
+    </geometry>
+  </collision>
+  <visual>
+    <geometry>
+      <mesh filename="package://rsy_robot_startup/meshes/cube_stand.stl" scale="0.001 0.001 0.001"/>
+    </geometry>
+    <material name="grey">
+      <color rgba="0.5 0.5 0.5 1.0"/>
+    </material>
+  </visual>
+</link>
+<joint name="world_to_cubestand" type="fixed">
+  <parent link="world"/>
+  <child link="cubestand"/>
+  <origin xyz="-0.15654 0.7294 0.0" rpy="0 0 0"/>
+</joint>
+<link name="cube_cubestand">
+  <collision>
+    <geometry>
+      <box size="0.06 0.06 0.06"/>
+    </geometry>
+  </collision>
+  <visual>
+    <geometry>
+      <box size="0.06 0.06 0.06"/>
+    </geometry>
     <material name="yellow">
       <color rgba="1.0 1.0 0.0 0.1"/>
@@ -313,7 +331,8 @@
   </visual>
 </link>
-<joint name="world_to_cube_stand" type="fixed">
-  <parent link="world"/>
-  <child link="cube_stand"/>
+<joint name="cubestand_to_cube_cubestand" type="fixed">
+  <parent link="cubestand"/>
+  <child link="cube_cubestand"/>
+  <origin xyz="0 0 0.172" rpy="0 0 0"/>
 </joint>
 <xacro:ur_robot
