Commit message: Add detailed planning session logs for January 13, 2026
- Introduced a new log file capturing multiple planning sessions.
- Each session includes input parameters, IK details, configuration settings, planning phases, results, execution details, and summaries.
- Captured various scenarios including successful and failed attempts, backtracking events, and execution durations for different motion steps and robot configurations.

File: src/rsy_robot_startup/config/ur.urdf.xacro (robot description, xacro)
@@ -314,5 +314,5 @@
   <parent link="world"/>
   <child link="cubestand"/>
-  <origin xyz="-0.15654 0.7294 0.0" rpy="0 0 0"/>
+  <origin xyz="-0.11854 0.7334 0.0" rpy="0 0 0"/>
 </joint>
 <link name="cube_cubestand">
@@ -335,4 +335,84 @@
   <child link="cube_cubestand"/>
   <origin xyz="0 0 0.172" rpy="0 0 0"/>
+</joint>
+<link name="finger_1_robot1">
+  <collision>
+    <geometry>
+      <box size="0.022 0.015 0.05"/>
+    </geometry>
+  </collision>
+  <visual>
+    <geometry>
+      <box size="0.022 0.015 0.05"/>
+    </geometry>
+    <material name="red">
+      <color rgba="1.0 0.0 0.0 0.1"/>
+    </material>
+  </visual>
+</link>
+<joint name="robot1_tcp_to_finger_1_robot1" type="fixed">
+  <parent link="robot1_tcp"/>
+  <child link="finger_1_robot1"/>
+  <origin xyz="0.0535 0 -0.065" rpy="0 0 0"/>
+</joint>
+<link name="finger_2_robot1">
+  <collision>
+    <geometry>
+      <box size="0.022 0.015 0.05"/>
+    </geometry>
+  </collision>
+  <visual>
+    <geometry>
+      <box size="0.022 0.015 0.05"/>
+    </geometry>
+    <material name="red">
+      <color rgba="1.0 0.0 0.0 0.1"/>
+    </material>
+  </visual>
+</link>
+<joint name="robot1_tcp_to_finger_2_robot1" type="fixed">
+  <parent link="robot1_tcp"/>
+  <child link="finger_2_robot1"/>
+  <origin xyz="-0.0535 0 -0.065" rpy="0 0 0"/>
+</joint>
+<link name="finger_1_robot2">
+  <collision>
+    <geometry>
+      <box size="0.022 0.015 0.05"/>
+    </geometry>
+  </collision>
+  <visual>
+    <geometry>
+      <box size="0.022 0.015 0.05"/>
+    </geometry>
+    <material name="red">
+      <color rgba="1.0 0.0 0.0 0.1"/>
+    </material>
+  </visual>
+</link>
+<joint name="robot2_tcp_to_finger_1_robot2" type="fixed">
+  <parent link="robot2_tcp"/>
+  <child link="finger_1_robot2"/>
+  <origin xyz="0.0535 0 -0.065" rpy="0 0 0"/>
+</joint>
+<link name="finger_2_robot2">
+  <collision>
+    <geometry>
+      <box size="0.022 0.015 0.05"/>
+    </geometry>
+  </collision>
+  <visual>
+    <geometry>
+      <box size="0.022 0.015 0.05"/>
+    </geometry>
+    <material name="red">
+      <color rgba="1.0 0.0 0.0 0.1"/>
+    </material>
+  </visual>
+</link>
+<joint name="robot2_tcp_to_finger_2_robot2" type="fixed">
+  <parent link="robot2_tcp"/>
+  <child link="finger_2_robot2"/>
+  <origin xyz="-0.0535 0 -0.065" rpy="0 0 0"/>
 </joint>
 <xacro:ur_robot
